Commit message: Small tweaks to get URDF to render properly.

File: data/urdf/inertiabot3.urdf (robot description, URDF)
Before this commit: robot inertiabot3, 3 links, 2 joints
Links:
- link body: mass 1.0 -> 0.2102; geometry collision box size=0.130 0.030 0.070; visual mesh filename=inertiabot3_description/robot_sim_body.dae scale=0.001 0.001 0.001
- link leg_A: mass 1.0 -> 0.1202; geometry collision box size=0.100 0.030 0.070; visual mesh filename=inertiabot3_description/robot_sim_leg.dae scale=0.001 0.001 0.001
- link leg_B: geometry collision box size=0.100 0.030 0.070; visual mesh filename=inertiabot3_description/robot_sim_leg.dae scale=0.001 0.001 0.001
Joints:
- joint HipA: axis 0 1 0 -> 0 0 1; limit (none) -> lower=-1.57079632679 upper=1.57079632679 effort=10 velocity=1.0; origin xyz=0.0 0.0 -0.125 rpy=0.0 0.0 0.0 -> xyz=-0.056 0.0 0.0 rpy=0.0 0.0 0.0
- joint HipB: axis 0 1 0 -> 0 0 1; limit (none) -> lower=-1.57079632679 upper=1.57079632679 effort=10 velocity=1.0; origin xyz=0.0 0.0 0.125 rpy=0.0 0.0 0.0 -> xyz=0.056 0.0 0.0 rpy=0.0 0.0 0.0

Commit message: inertiabot3 now has a URDF description and an XML scriptable control

File: data/urdf/inertiabot3.urdf (robot description, URDF)
Before this commit: robot inertiabot3, 3 links, 2 joints
Links:
- link body: geometry collision box size=0.085 0.030 0.070; visual mesh filename=inertiabot3_description/robot_sim_body.dae scale=0.001 0.001 0.001
- link leg_A: geometry collision box size=0.085 0.030 0.070; visual mesh filename=inertiabot3_description/robot_sim_leg.dae scale=0.001 0.001 0.001
- link leg_B: mass 1.0 -> 0.1202; geometry collision box size=0.085 0.030 0.070; visual mesh filename=inertiabot3_description/robot_sim_leg.dae scale=0.001 0.001 0.001
